Commit message: add the Gazebo world launch package

File: my_rb1_description/urdf/my_rb1_robot.urdf (robot description, URDF)
Before this commit: robot rb1_robot, 7 links, 6 joints
Links:
- link left_wheel: geometry collision cylinder length=0.03 radius=0.025; visual cylinder length=0.03 radius=0.025
- link right_wheel: geometry collision cylinder length=0.03 radius=0.025; visual cylinder length=0.03 radius=0.025

Commit message: add the Gazebo plugins

File: my_rb1_description/urdf/my_rb1_robot.urdf (robot description, URDF)
Before this commit: robot rb1_robot, 7 links, 6 joints
Joints:
- joint base_link_left_wheel_joint: axis (none) -> 0 1 0
- joint base_link_right_wheel_joint: axis (none) -> 0 1 0
